File: esphome-rf-doorbell.kicad_sch (KiCad schematic)
At the start: 58 parts, among them J1 B4B-XH, J2 CONUFL001-SMD-T, J3 PROG, SW1 Boot, U1 ESP32-S2-MINI-2, U2 RFM95W-868S2, U3 TLP2391, U4 G3VM-63ER, U5 MP5493GJ-Z, U6 ASSR-1218

Commit message: Replace RF module, finish routing
Parts:
- removed J3: PROG, TestPoint:TestPoint_2Pads_Pitch2.54mm_Drill0.8mm, symbol Connector_Generic:Conn_01x02
- removed JP3: SolderJumper_2_Open, Jumper:SolderJumper-2_P1.3mm_Open_RoundedPad1.0x1.5mm, symbol Jumper:SolderJumper_2_Open
- removed U2: RFM95W-868S2, RF_Module:HOPERF_RFM9XW_SMD, symbol RF_Module:RFM95W-868S2
- added C6: 0.1uF, Capacitor_SMD:C_0402_1005Metric, symbol Device:C
- added J3, J4: Conn_01x01, TestPoint:TestPoint_Keystone_5000-5004_Miniature, symbol Connector_Generic:Conn_01x01
- added U2: RFM69W, RF_Module:HOPERF_RFM69HW, symbol RF_Module:RFM69W
- U3: renamed from U6; value ASSR-1218 -> G3VM-31DR; footprint Package_SO:SO-4_4.4x4.3mm_P2.54mm -> Package_DIP:SMDIP-4_W7.62mm
- renumbered C6 to C1, C13 to C10, C8 to C11, C9 to C12, C11 to C13, C10 to C14, C5 to C2, C4 to C3, C3 to C4, C7 to C5, C1 to C7, C2 to C8, C12 to C9, D2 to D1, D1 to D2, D6 to D4, D4 to D6, JP4 to JP1, JP1 to JP3, L2 to L1, L1 to L2, R16 to R10, R7 to R11, R8 to R12, R12 to R13, R11 to R14, R10 to R15, R9 to R16, R5 to R2, R2 to R3, R6 to R4, R3 to R5, R4 to R6, R13 to R7, R14 to R8, R15 to R9, U5 to U1, U1 to U4, U4 to U5, U3 to U6
Connections:
- net +3.3V: now also C3.1, C4.1, L1.2, R2.1, C6.1, U2.8 (3.3V)
- net BELL_OFF: now also U4.16 (IO12); no longer U4.20 (IO16)
- net GND: now also C6.2, U2.11 (GND), U2.9 (GND)
- net OPEN_BUZZER: now also U4.18 (IO14); no longer U4.19 (IO15)
- net RF.Antenna: now also U2.10 (ANA)
- net RF.CE: now also U4.15 (IO11), U2.15 (NSS); no longer U4.14 (IO10)
- net RF.MISO: now also U2.13 (MISO)
- net RF.MOSI: now also U4.14 (IO10), U2.14 (MOSI); no longer U4.15 (IO11)
- net RF.Reset: now also U4.11 (IO7), U2.1 (RESET); no longer U4.17 (IO13)
- net RF.SCLK: now also U4.12 (IO8), U2.12 (SCK); no longer U4.16 (IO12)
- net UART_RX: now also J4.1 (Pin_1)
- net UART_TX: now also J3.1 (Pin_1)
- net ~{BELL_SIGNAL}: now also U4.17 (IO13); no longer U4.18 (IO14)
- net RF.IO0: now reaches U4.10 (IO6)
- net RF.IO0: now also U2.2 (DIO0)
- net at U4.4 (IO0): now also SW1.2
- net RF.IO5: now reaches U4.5 (IO1)
- net RF.IO5: now also U2.7 (DIO5)
- net RF.IO4: now reaches U4.6 (IO2)
- net RF.IO4: now also U2.6 (DIO4)
- net RF.IO3: now reaches U4.7 (IO3)
- net RF.IO3: now also U2.5 (DIO3)
- net RF.IO2: now reaches U4.8 (IO4)
- net RF.IO2: now also U2.4 (DIO2)
- net RF.IO1: now reaches U4.9 (IO5)
- net RF.IO1: now also U2.3 (DIO1)
- net ~{POWER_FAIL}: now reaches U1.2 (PFAIL)
- net ~{POWER_FAIL}: now also U4.19 (IO15)
- net EN: no longer names the net of C9.1, R7.2, U4.45 (EN)
- net EN: no longer SW1.2
- no-connect marks 7 -> 22
Other:
- moved on the sheet: C5, C9, R7, SW1
