File: remote/remote.kicad_pcb (KiCad board)
At the start: 2 copper layers, 35.4 x 24.4 mm, 11 parts, among them J1 Conn_Coaxial, SW1 SW_SPST, U1 RFM69W, U2 PIC12LF1501-xMS

Commit message: Fix ERC
Parts:
- U2: value PIC12LF1501-xMS -> PIC12LF1552
Changed lines of the file:
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@@
 			)
 		)
-		(property "Value" "PIC12LF1501-xMS"
+		(property "Value" "PIC12LF1552"
 			(at 0 2.45 0)
 			(layer "F.Fab")
@@
 			)
 		)
-		(property "Datasheet" "https://ww1.microchip.com/downloads/en/DeviceDoc/41615A.pdf"
+		(property "Datasheet" "https://ww1.microchip.com/downloads/aemDocuments/documents/OTH/ProductDocuments/DataSheets/40001674F.pdf"
 			(at 0 0 0)
 			(layer "F.Fab")

Commit message: Base board Rev3
Parts:
- removed J1: Conn_Coaxial, Connector_Coaxial:U.FL_Hirose_U.FL-R-SMT-1_Vertical
- added JP1: Jumper ~{MCLR}, Jumper:SolderJumper-2_P1.3mm_Open_RoundedPad1.0x1.5mm, F.Cu at (114.0, 78.2)
- added JP2: Jumper ICSPDAT, Jumper:SolderJumper-2_P1.3mm_Open_RoundedPad1.0x1.5mm, F.Cu at (115.5, 46.1)
- added JP3: Jumper ICSPCLK, Jumper:SolderJumper-2_P1.3mm_Open_RoundedPad1.0x1.5mm, F.Cu at (115.5, 42.8)
- added TP1: TestPoint, TestPoint:TestPoint_Keystone_5000-5004_Miniature, F.Cu at (118.5, 42.3)
- added TP2: TestPoint, TestPoint:TestPoint_Keystone_5000-5004_Miniature, F.Cu at (118.5, 45.7)
- added TP3: TestPoint, TestPoint:TestPoint_Keystone_5000-5004_Miniature, F.Cu at (118.6, 74.7)
- added TP4: TestPoint, TestPoint:TestPoint_Keystone_5000-5004_Miniature, F.Cu at (89.6, 76.6)
- C1, C2, C4: footprint Capacitor_SMD:C_0402_1005Metric_Pad0.74x0.62mm_HandSolder -> Capacitor_SMD:C_0603_1608Metric_Pad1.08x0.95mm_HandSolder
- R1: value R -> 1k; footprint Resistor_SMD:R_0402_1005Metric_Pad0.72x0.64mm_HandSolder -> Resistor_SMD:R_0603_1608Metric_Pad0.98x0.95mm_HandSolder
- R2: value R -> 10k; footprint Resistor_SMD:R_0402_1005Metric_Pad0.72x0.64mm_HandSolder -> Resistor_SMD:R_0603_1608Metric_Pad0.98x0.95mm_HandSolder
- moved C1 61.3 mm to (110.3, 59.0), turned to 0 degrees
- moved U2 55.4 mm to (111.7, 61.5), turned to 0 degrees
- moved R2 53.4 mm to (109.5, 72.9), turned to 180 degrees
- moved C4 50.0 mm to (112.9, 74.4), turned to 180 degrees
- moved C2 49.9 mm to (90.5, 59.7), turned to 90 degrees
- moved R1 49.4 mm to (112.9, 72.9), turned to 0 degrees
- moved SW1 49.0 mm to (111.3, 68.8), turned to -90 degrees
- moved U1 48.7 mm to (99.5, 68.6)
- moved C3 47.5 mm to (90.5, 63.1), turned to -90 degrees
- moved BT1 47.1 mm to (104.5, 68.5)
Connections:
- U1 pad 10: Net-(J1-In) -> unconnected-(U1-ANA-Pad10)
- U2 pad 4: /BTN -> Net-(JP1-A)
- U2 pad 6: /SCK -> Net-(JP3-B)
- U2 pad 7: /SDO -> Net-(JP2-B)
Routing:
- net VDD: track 0.00 -> 39.3 mm, vias 0 -> 2
- net /RFINT: track 0.00 -> 6.48 mm
- net GND: track 0.00 -> 0.27 mm, vias 0 -> 11
- added copper zone on B.Cu, net GND
- added copper zone on F.Cu, net GND
Other:
- board size 35.4 x 24.4 mm -> 33.1 x 21.7 mm
- board text added: "GND"
