File: base/esphome-rf-doorbell.kicad_sch (KiCad schematic)
At the start: 80 parts, among them J1 PTSM 0,5/ 4-2,5-H SMD R24, J2 Conn_01x06, Q1 PMZB390UNE, SW1 Flash, SW2 CL-SB-22A-11T, U1 ESP32-C6-MINI-1, U2 Wio-SX1262, U3 ISL23315, U4 MAX17260, U5 LTC4079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

Commit message: Update docs, fix fuel gauge issue
Parts:
- BT1: value ~ -> (none)

Commit message: Rev 4
Parts:
- added R24: 47k, Capacitor_SMD:C_0402_1005Metric, symbol Device:R_Small
- added R25: 0, Capacitor_SMD:C_0402_1005Metric, symbol Device:R_Small
- added R26: 100k, Capacitor_SMD:C_0402_1005Metric, symbol Device:R_Small
- R11: value 30k -> 20k
- R15, R16: symbol Device:R -> Device:R_Small
Connections:
- net +3.3V: now also R24.1, R26.1
- net at U2.1 (RF_SW1): now also R25.2
- net RF_SWITCH: now reaches U1.20 (IO15)
- net RF_SWITCH: now also R25.1, R26.2
- net at U1.22 (IO8): now also R24.2
- no-connect marks 10 -> 7
Other:
- moved on the sheet: C18, D2, D3, D5, JP1, JP2, JP4, R15, R16, R18, R19, R2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
